File: electronique/mainBoard.brd (EAGLE design)
At the start: 63 x 67.5 mm, 38 parts, among them IC1 L298, IC2 7805TV

Commit message: control des moteurs OK + controle tension des lipos fonctionnel
Connections:
- net ENABLE_DROIT: now also IC1.6, U$1.0; no longer IC1.11, U$1.1
- net ENABLE_GAUCHE: now also IC1.11, U$1.1; no longer IC1.6, U$1.0
- net IN1_DROIT: now also IC1.5, U$1.23/A9; no longer IC1.10, U$1.21/A7
- net IN1_GAUCHE: now also IC1.10, U$1.21/A7; no longer IC1.5, U$1.23/A9
- net IN2_DROIT: now also IC1.7, U$1.22/A8; no longer IC1.12, U$1.20/A6
- net IN2_GAUCHE: now also IC1.12, U$1.20/A6; no longer IC1.7, U$1.22/A8
Routing:
- net IN2_GAUCHE: track 9.17 -> 69.4 mm, vias 1 -> 6
- net IN2_DROIT: track 69.4 -> 9.17 mm, vias 6 -> 1
- net ENABLE_GAUCHE: track 55.9 -> 35.8 mm, vias 4 -> 1
- net ENABLE_DROIT: track 35.8 -> 55.9 mm, vias 1 -> 4
- net IN1_GAUCHE: track 8.64 -> 22.0 mm
- net IN1_DROIT: track 22.0 -> 8.64 mm
Changed lines of the file:
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@@
 <layer number="45" name="Holes" color="7" fill="1" visible="no" active="yes"/>
 <layer number="46" name="Milling" color="3" fill="1" visible="no" active="yes"/>
-<layer number="47" name="Measures" color="7" fill="1" visible="no" active="yes"/>
-<layer number="48" name="Document" color="7" fill="1" visible="no" active="yes"/>
-<layer number="49" name="Reference" color="7" fill="1" visible="no" active="yes"/>
-<layer number="51" name="tDocu" color="7" fill="1" visible="no" active="yes"/>
-<layer number="52" name="bDocu" color="7" fill="1" visible="no" active="yes"/>
+<layer number="47" name="Measures" color="7" fill="1" visible="yes" active="yes"/>
+<layer number="48" name="Document" color="7" fill="1" visible="yes" active="yes"/>
+<layer number="49" name="Reference" color="7" fill="1" visible="yes" active="yes"/>
+<layer number="51" name="tDocu" color="7" fill="1" visible="yes" active="yes"/>
+<layer number="52" name="bDocu" color="7" fill="1" visible="yes" active="yes"/>
 <layer number="90" name="Modules" color="5" fill="1" visible="no" active="yes"/>
 <layer number="91" name="Nets" color="2" fill="1" visible="no" active="no"/>
@@
 <wire x1="46.99" y1="16.51" x2="48.895" y2="14.605" width="0.2032" layer="1"/>
 </signal>
-<signal name="ENABLE_GAUCHE">
+<signal name="ENABLE_DROIT">
 <contactref element="IC1" pad="6"/>
 <contactref element="U$1" pad="0"/>
@@
 <via x="30.48" y="41.91" extent="1-16" drill="0.6096"/>
 </signal>
-<signal name="ENABLE_DROIT">
+<signal name="ENABLE_GAUCHE">
 <contactref element="IC1" pad="11"/>
 <contactref element="U$1" pad="1"/>
@@
 <via x="16.51" y="43.18" extent="1-16" drill="0.6096"/>
 </signal>
-<signal name="IN1_GAUCHE">
+<signal name="IN1_DROIT">
 <contactref element="IC1" pad="5"/>
 <contactref element="U$1" pad="23/A9"/>
@@
 <wire x1="31.115" y1="40.005" x2="31.73" y2="40.62" width="0.2032" layer="16"/>
 </signal>
-<signal name="IN2_GAUCHE">
+<signal name="IN2_DROIT">
 <contactref element="IC1" pad="7"/>
 <contactref element="U$1" pad="22/A8"/>
@@
 <via x="28.575" y="36.83" extent="1-16" drill="0.6096"/>
 </signal>
-<signal name="IN1_DROIT">
+<signal name="IN1_GAUCHE">
 <contactref element="IC1" pad="10"/>
 <contactref element="U$1" pad="21/A7"/>
@@
 <wire x1="36.83" y1="33.655" x2="36.81" y2="34.27" width="0.2032" layer="16"/>
 </signal>
-<signal name="IN2_DROIT">
+<signal name="IN2_GAUCHE">
 <contactref element="IC1" pad="12"/>
 <contactref element="U$1" pad="20/A6"/>
